File: PCB/PCB_copy_rachel/WallNet_Main/WallNet_Main.kicad_pcb (KiCad board)
At the start: 4 copper layers, 120.6 x 69.8 mm, 87 parts, among them J1 Conn_01x05_Pin, J101 usbc_plug_lfg, J102 01x04 Molex, J201 01x04 Molex, J202 Conn_01x07_Socket, J203 02x12 Connector, Q201 BSS138, SW1 SW, U1 BT832, U101 BQ25895RTWT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

Commit message: added power and fixed errors
Routing:
- net VDD_nrf: track 18.3 -> 60.4 mm, vias 0 -> 26
- net GND: track 4.50 -> 23.5 mm, vias 0 -> 10
- net /Sensors/VDHR: track 1.71 -> 7.37 mm, vias 1 -> 2
- removed copper zone on In2.Cu, net VDD_nrf
Other:
- board size 120.6 x 69.8 mm -> 120.7 x 70.2 mm
