File: PCB/WallNet_Main/Sensors_WallNet.kicad_sch (KiCad schematic)
At the start: 43 parts, among them J2 Conn_01x05_Pin, J201 01x04 Molex, J203 02x12 Connector, Q201 BSS138, U201 CPT-9019B-SMT-TR, U202 SAM-M10Q-00B

Commit message: Redid PCB still need to DRC the design
Parts:
- removed TP201: TS_TX, 5001:KEYSTONE_5001, symbol Connector:TestPoint
- removed TP202: TS_RX, 5001:KEYSTONE_5001, symbol Connector:TestPoint
- removed TP203: GPS_SDA, 5001:KEYSTONE_5001, symbol Connector:TestPoint
- removed TP204: GPS_SCL, 5001:KEYSTONE_5001, symbol Connector:TestPoint
- removed TP205: GPS_INT, 5001:KEYSTONE_5001, symbol Connector:TestPoint
- removed TP206: GPS_TP, 5001:KEYSTONE_5001, symbol Connector:TestPoint
- removed TP207: RFID_SCL, 5001:KEYSTONE_5001, symbol Connector:TestPoint
- removed TP208: RFID_SDA, 5001:KEYSTONE_5001, symbol Connector:TestPoint
- removed TP209: RFID_GPO, 5001:KEYSTONE_5001, symbol Connector:TestPoint
- removed TP210: EP_DC, 5001:KEYSTONE_5001, symbol Connector:TestPoint
- removed TP211: EP_SDA, 5001:KEYSTONE_5001, symbol Connector:TestPoint
- removed TP212: EP_SCL, 5001:KEYSTONE_5001, symbol Connector:TestPoint
- removed TP213: EP_CSB, 5001:KEYSTONE_5001, symbol Connector:TestPoint
- removed TP214: EP_BUSY, 5001:KEYSTONE_5001, symbol Connector:TestPoint
- removed TP215: EP_RESET, 5001:KEYSTONE_5001, symbol Connector:TestPoint
- added R206: 10k, Resistor_SMD:R_0603_1608Metric, symbol Device:R_Small_US
- renumbered J2 to J202
Connections:
- net Buzzer: now also R206.1
- net GND: now also R206.2
- net VGL: now also D202.2 (A); no longer D202.1 (K)
- net at C211.2, D203.2 (A): now also D202.1 (K); no longer D202.2 (A)
- net EP_SDA renamed EP_DIN
Other:
- note removed: "Implement Backup circuit (Socket connector)"
- note removed: "Test Points"
- moved on the sheet: D202
